File: hardware/Baja Pro v4.kicad_sch (KiCad schematic)
At the start: 24 parts, among them P1 Header-Female-2.54_1x4, P2 Header-Female-2.54_1x2, P4 Header-Female-2.54_1x6, U1 FM24CL04B-GTR_C365762, U2 DC-DC stepdown, U3 AMS1117-3.3, U4 Thermistor, X1 ESP32_WROOM32

Commit message: Update to KiCAD9 Create missing symbols Replace symbols with KiCAD symbols Link symbols with footprints
Signed-off-by: Ilias Daradimos <judgedrid@gmail.com>
Parts:
- removed .: NO, symbol Unknown_816_574
- removed X1: ESP32_WROOM32, symbol Unknown_850_940
- added U4: ESP32-WROOM-32, RF_Module:ESP32-WROOM-32, symbol RF_Module:ESP32-WROOM-32
- C1: footprint (none) -> Baja Pro v4:1206; symbol Cap_1206_EU -> Device:C; Manufacturer Part ? -> (none)
- C2: footprint (none) -> Baja Pro v4:1206; symbol Cap_1206_EU_1 -> Device:C; Manufacturer Part ? -> (none)
- C3: footprint (none) -> Baja Pro v4:1206; symbol Cap_1206_EU_2 -> Device:C; Manufacturer Part ? -> (none)
- C4: footprint (none) -> Baja Pro v4:1206; symbol Cap_1206_EU_3 -> Device:C; Manufacturer Part ? -> (none)
- C5: footprint (none) -> Baja Pro v4:1206; symbol Cap_1206_EU_4 -> Device:C; Manufacturer Part ? -> (none)
- C6: footprint (none) -> Baja Pro v4:1206; symbol 1206B226K160NT -> Device:C
- D1: footprint (none) -> Diode_SMD:D_SOD-123F; symbol Unknown_255_175 -> Device:D; Manufacturer Hottech -> (none); Manufacturer Part 1N4007 -> (none); Supplier LCSC -> (none); Supplier Part C181127 -> (none)
- GPS1: footprint (none) -> Baja Pro v4:GY-NEO6MV2; symbol Unknown_1385_195 -> BajaPro:GY-NEO6MV2
- J1: renamed from U4; footprint (none) -> Connector_PinHeader_2.54mm:PinHeader_1x02_P2.54mm_Vertical; symbol Unknown_1506_957 -> Connector_Generic:Conn_01x02; Manufacturer Part ? -> (none)
- LCD1: footprint (none) -> Baja Pro v4:ERC12864-655; symbol Unknown_155_837 -> BajaPro:ERC12864-655
- P1: value Header-Female-2.54_1x4 -> Remote; footprint (none) -> Connector_PinHeader_2.54mm:PinHeader_1x04_P2.54mm_Vertical; symbol Unknown_1469_705 -> Connector_Generic:Conn_01x04; Manufacturer ReliaPro -> (none); Manufacturer Part Header-Female-2.54_1x4 -> (none); Supplier LCSC -> (none); Supplier Part C124413 -> (none)
- P2: value Header-Female-2.54_1x2 -> Power; footprint (none) -> Connector_PinHeader_2.54mm:PinHeader_1x02_P2.54mm_Vertical; symbol Unknown_130_190 -> Connector_Generic:Conn_01x02; Manufacturer BOOMELE -> (none); Manufacturer Part 2.54-1*2PFemale -> (none); Supplier LCSC -> (none); Supplier Part C49661 -> (none)
- P4: value Header-Female-2.54_1x6 -> Flash; footprint (none) -> Connector_PinHeader_2.54mm:PinHeader_1x06_P2.54mm_Vertical; symbol Unknown_1465_500 -> Connector_Generic:Conn_01x06; Manufacturer BOOMELE -> (none); Manufacturer Part Female header 1*6p -> (none); Supplier LCSC -> (none); Supplier Part C40877 -> (none)
- R1: footprint (none) -> Baja Pro v4:1206; symbol Res_1206(1/4W)_EU -> Device:R; Manufacturer Part ? -> (none)
- R2: footprint (none) -> Baja Pro v4:1206; symbol Res_1206(1/4W)_EU_1 -> Device:R; Manufacturer Part ? -> (none)
- R3: footprint (none) -> Baja Pro v4:1206; symbol Res_1206(1/4W)_EU_2 -> Device:R; Manufacturer Part ? -> (none)
- R4: footprint (none) -> Baja Pro v4:1206; symbol Res_1206(1/4W)_EU_3 -> Device:R; Manufacturer Part ? -> (none)
- R5: footprint (none) -> Baja Pro v4:1206; symbol Res_1206(1/4W)_EU_4 -> Device:R; Manufacturer Part ? -> (none)
- R6: footprint (none) -> Baja Pro v4:1206; symbol Res_1206(1/4W)_EU_5 -> Device:R; Manufacturer Part ? -> (none)
- U1: footprint (none) -> Baja Pro v4:SOIC-8_150MIL; symbol Unknown_785_200 -> BajaPro:FM24CL04B-GTR_C365762
- U2: footprint (none) -> Baja Pro v4:DC-DC STEPDOWN; symbol Unknown_365_205 -> BajaPro:DC-DC Stepdown
- U3: footprint (none) -> Package_TO_SOT_SMD:SOT-223-3_TabPin2; symbol Unknown_255_375 -> Regulator_Linear:AMS1117-3.3; Manufacturer AMS -> (none); Manufacturer Part AMS1117-3.3 -> (none); Supplier LCSC -> (none); Supplier Part C6186 -> (none)
Connections:
- net 3V3: now also U4.2 (VDD)
- net 5V: now also J1.2 (Pin_2), U3.3 (VI); no longer J1.1 (THERM_1), U3.1 (In)
- net DISPLAY_BL: now also U4.11 (IO26)
- net DISPLAY_CD: now also U4.10 (IO25)
- net DISPLAY_CS: now also U4.13 (IO14)
- net DISPLAY_DATA: now also U4.14 (IO12)
- net DISPLAY_RST: now also U4.12 (IO27)
- net DISPLAY_SCLK: now also U4.16 (IO13)
- net FLASH_DTR: now also U4.25 (IO0)
- net FLASH_RTS: now also U4.3 (EN)
- net FLASH_RX: now also U4.34 (RXD0/IO3)
- net FLASH_TX: now also U4.35 (TXD0/IO1)
- net GND: now also U3.1 (GND), U4.1 (GND), U4.15 (GND), U4.38 (GND), U4.39 (GND); no longer U1.1 (NC), U3.3 (GND)
- net GPS_RX: now also U4.28 (IO17)
- net GPS_TX: now also U4.27 (IO16)
- net MEM_SCL: now also U4.36 (IO22)
- net MEM_SDA: now also U4.33 (IO21)
- net R_NEXT: now also U4.6 (IO34)
- net R_PREV: now also U4.8 (IO32)
- net R_SELECT: now also U4.9 (IO33)
- net TEMP: now also J1.1 (Pin_1), U4.23 (IO15); no longer J1.2 (THERM_2)
- net at D1.1 (K): now also U2.2 (In+); no longer P2.2
- net at D1.2 (A): now also P2.2 (Pin_2); no longer U2.2 (In+)
- no-connect marks 16 -> 15
Other:
- title: (none) -> Baja Pro v4
